File: SWD-Breakout/SWD-Breakout.kicad_pcb (KiCad board)
At the start: 2 copper layers, 19.1 x 15.2 mm, 2 parts, among them J1 Conn_02x05_Odd_Even, J2 Conn_01x04

Commit message: SWD Breakout updates
Parts:
- added G***: LOGO, Images:amber, B.Cu at (144.1, 81.3)
Other:
- board text added: "David Richmond"
- board text added: "dave@prstat.org"
