File: M68K-Nucleo/M68K-Nucleo.sch (KiCad schematic (older format))
At the start: 18 parts, among them J1 VSel, J2 Current Sense, J3 Conn_01x04, U1 68000D, U2 NUCLEO144-F746ZG, U3 TXB0104D

Commit message: Changed level shifter package on M68k board
Parts:
- U3: footprint Package_SO:SOIC-14_3.9x8.7mm_P1.27mm -> Package_SO:TSSOP-14_4.4x5mm_P0.65mm
Changed lines of the file:
@@
 F 0 "U3" H 7150 4111 50  0000 C CNN
 F 1 "TXB0104D" H 7150 4020 50  0000 C CNN
-F 2 "Package_SO:SOIC-14_3.9x8.7mm_P1.27mm" H 7150 4150 50  0001 C CNN
+F 2 "Package_SO:TSSOP-14_4.4x5mm_P0.65mm" H 7150 4150 50  0001 C CNN
 F 3 "http://www.ti.com/lit/ds/symlink/txb0104.pdf" H 7260 4995 50  0001 C CNN
 	1    7150 4900
