File: ESP32-D1Mini-HUB75/ESP32-D1Mini-HUB75.sch (KiCad schematic (older format))
At the start: 5 parts, among them J1 Conn_01x02, J2 Conn_01x02, J3 Conn_01x02, J4 Conn_02x08_Odd_Even, U1 mini_esp32

Commit message: updated screw terminal in esp32 hub75 board to use 8.5mm terminal that better suits the power cable that comes with the matrices
Parts:
- J1: footprint TerminalBlock_Dinkle:TerminalBlock_Dinkle_DT-55-B01X-02_P10.00mm -> ESP32-D1Mini-HUB75:KF8500-2P
Changed lines of the file:
@@
 F 0 "J1" H 6880 1342 50  0000 L CNN
 F 1 "Conn_01x02" H 6880 1251 50  0000 L CNN
-F 2 "TerminalBlock_Dinkle:TerminalBlock_Dinkle_DT-55-B01X-02_P10.00mm" H 6800 1350 50  0001 C CNN
+F 2 "ESP32-D1Mini-HUB75:KF8500-2P" H 6800 1350 50  0001 C CNN
 F 3 "~" H 6800 1350 50  0001 C CNN
 	1    6800 1350
