File: Gotek-PS2/Gotek-PS2.kicad_pcb (KiCad board)
At the start: 2 copper layers, 52 parts, among them J1 Conn_01x02, J2 Conn_01x02, J3 Conn_01x02, J4 Conn_02x17_Odd_Even, J5 Conn_02x17_Odd_Even, J6 Conn_01x04

Commit message: Missed gotek updates
Parts:
- added G***: LOGO, Images:amber, F.Cu at (129.3, 107.4)
- added svg2mod: G***, label, F.Cu at (84.1, 65.5)
- added svg2mod: G***, label, F.Cu at (100.3, 90.4)
- added svg2mod: G***, label, F.Cu at (95.2, 93.2)
- added svg2mod: G***, label, F.Cu at (100.3, 95.8)
- added svg2mod: G***, label, F.Cu at (95.2, 98.3)
- added svg2mod: G***, label, F.Cu at (100.3, 101.1)
- added svg2mod: G***, label, F.Cu at (95.2, 103.4)
- added svg2mod: G***, label, F.Cu at (100.3, 105.9)
- added svg2mod: G***, label, F.Cu at (94.7, 108.5)
- added svg2mod: G***, label, F.Cu at (106.9, 105.9)
- added svg2mod: G***, label, F.Cu at (106.9, 100.8)
- added svg2mod: G***, label, F.Cu at (145.5, 62.2)
- added svg2mod: G***, label, F.Cu at (106.7, 95.8)
- added svg2mod: G***, label, F.Cu at (106.7, 90.7)
- added svg2mod: G***, label, F.Cu at (106.9, 85.6)
- added svg2mod: G***, label, F.Cu at (106.9, 80.5)
- added svg2mod: G***, label, F.Cu at (106.9, 75.4)
- added svg2mod: G***, label, F.Cu at (106.9, 70.4)
- added svg2mod: G***, label, F.Cu at (112.0, 67.8)
- added svg2mod: G***, label, F.Cu at (112.0, 72.9)
- added svg2mod: G***, label, F.Cu at (112.0, 78.0)
- added svg2mod: G***, label, F.Cu at (112.0, 83.1)
- added svg2mod: G***, label, F.Cu at (96.3, 67.3)
- added svg2mod: G***, label, F.Cu at (112.0, 88.1)
- added svg2mod: G***, label, F.Cu at (112.0, 93.2)
- added svg2mod: G***, label, F.Cu at (112.0, 98.3)
- added svg2mod: G***, label, F.Cu at (112.0, 103.4)
- added svg2mod: G***, label, F.Cu at (112.0, 108.5)
- added svg2mod: G***, label, F.Cu at (100.3, 75.4)
- added svg2mod: G***, label, F.Cu at (95.0, 78.0)
- added svg2mod: G***, label, F.Cu at (100.3, 80.5)
- added svg2mod: G***, label, F.Cu at (95.2, 83.1)
- added svg2mod: G***, label, F.Cu at (100.3, 85.6)
- added svg2mod: G***, label, F.Cu at (95.2, 88.1)
Routing:
- net GND: track 330.7 -> 47.4 mm, vias 0 -> 26
- net Net-(J2-Pad1): track 0.00 -> 82.6 mm, vias 0 -> 1
- net Net-(J3-Pad1): track 0.00 -> 79.6 mm, vias 0 -> 2
- net Net-(J1-Pad1): track 0.00 -> 71.2 mm
- net Net-(J2-Pad2): track 0.00 -> 67.7 mm, vias 0 -> 1
- net Net-(J1-Pad2): track 0.00 -> 62.2 mm, vias 0 -> 1
- net +5V: track 0.00 -> 58.3 mm
- net /Track0: track 0.00 -> 47.5 mm
- net /Direction: track 0.00 -> 47.5 mm
- net /DiskChg: track 0.00 -> 47.4 mm
- net /RData: track 0.00 -> 47.4 mm
- net /WData: track 0.00 -> 47.3 mm
- net /Step: track 0.00 -> 42.4 mm
- net /WPT: track 0.00 -> 42.4 mm
- net /WEn: track 0.00 -> 42.3 mm
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- added copper zone on B.Cu, net GND
Other:
- board outline added: 77.2 x 63 mm
- net class Power added: clearance 0.2, trace_width 0.5, via_dia 1, via_drill 0.6
- board text added: "12V"
- board text added: "5V"
- board text added: "GND"
- board text added: "d@verichmond.dev"
- board text removed: "GoTek"
- board text removed: "PS/2 Cable"
