File: Sun-KBD-Interface/Sun-KBD-Interface.kicad_pcb (KiCad board)
At the start: 2 copper layers, 88.9 x 57.1 mm, 93 parts, among them J1 Conn_01x08_Male, J10 Conn_01x04_Female, J2 Conn_01x05_Female, J3 Conn_01x05_Female, J4 Conn_01x05_Female, J5 Conn_01x05_Female, J6 Mini-DIN-8, J7 Mini-DIN-6, J8 Mini-DIN-6, J9 Conn_01x04_Female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

Commit message: Misc missed changes? Been a while since I really looked
Parts:
- added kibuzzard-13: G***, kibuzzard-6300B361, B.Cu at (110.5, 74.9)
- added kibuzzard-15: G***, kibuzzard-6300B3DE, B.Cu at (115.6, 64.8)
- added kibuzzard-18: G***, kibuzzard-6300B3ED, B.Cu at (115.6, 71.8)
- added kibuzzard-63B4EFA4: G***, kibuzzard-63B4EFA4, B.Cu at (110.5, 59.7)
- added kibuzzard-63B4EFB4: G***, kibuzzard-63B4EFB4, B.Cu at (110.5, 62.2)
- added kibuzzard-63B4F027: G***, kibuzzard-63B4F027, B.Cu at (110.5, 72.4)
- added kibuzzard-63B4F027: G***, kibuzzard-63B4F027, B.Cu at (110.5, 67.3)
- added kibuzzard-63B4F037: G***, kibuzzard-63B4F037, B.Cu at (110.5, 64.8)
- added kibuzzard-63B4F037: G***, kibuzzard-63B4F037, B.Cu at (110.5, 69.8)
- added kibuzzard-9: G***, kibuzzard-6300B31A, B.Cu at (110.5, 77.5)
