File: VideoIO/VideoIO.kicad_pcb (KiCad board)
At the start: 2 copper layers, 56 parts, among them J1 DB15_Male_HighDensity, J2 DB15_Male_HighDensity, J3 Conn_02x06_Odd_Even, J4 Conn_02x20_Odd_Even, U1 AMS1117, U2 AMS1117, U3 TVP7002

Commit message: More work on video io board
Parts:
- added C28: C, Capacitor_SMD:C_0805_2012Metric_Pad1.15x1.40mm_HandSolder, F.Cu at (101.1, 57.7)
- added C29: C, Capacitor_SMD:C_0805_2012Metric_Pad1.15x1.40mm_HandSolder, F.Cu at (100.8, 66.5)
- added C30: C, Capacitor_SMD:C_0805_2012Metric_Pad1.15x1.40mm_HandSolder, F.Cu at (100.8, 75.9)
- added JP1: Jumper, Connector_PinHeader_2.54mm:PinHeader_1x02_P2.54mm_Vertical, F.Cu at (97.0, 84.8)
- added JP2: Jumper, Connector_PinHeader_2.54mm:PinHeader_1x02_P2.54mm_Vertical, F.Cu at (94.0, 93.0)
- added R17: R, Resistor_SMD:R_0805_2012Metric_Pad1.15x1.40mm_HandSolder, F.Cu at (100.9, 78.9)
- added R18: R, Resistor_SMD:R_0805_2012Metric_Pad1.15x1.40mm_HandSolder, F.Cu at (100.8, 81.8)
- added U4: AMS1117, Package_TO_SOT_SMD:SOT-223-3_TabPin2, F.Cu at (93.7, 79.0)
- C1, C19, C2, C24, C3, C4, FB1, FB2, FB3, FB4, FB5, FB6: moved to B.Cu
- J3: footprint Connector_PinHeader_2.54mm:PinHeader_2x06_P2.54mm_Horizontal -> Connector_PinHeader_2.54mm:PinHeader_2x06_P2.54mm_Vertical
- J4: footprint Connector_PinHeader_2.54mm:PinHeader_2x20_P2.54mm_Horizontal -> Connector_PinHeader_2.54mm:PinHeader_2x20_P2.54mm_Vertical
- moved J4 73.7 mm to (142.3, 101.1), turned to 270 degrees
- moved C17 62.5 mm to (145.8, 36.3), turned to 270 degrees
- moved R12 62.4 mm to (174.2, 51.1)
- moved C14 61.6 mm to (139.4, 36.3), turned to 90 degrees
- moved C15 61.1 mm to (141.7, 36.3), turned to 90 degrees
- moved R1 56.3 mm to (101.1, 60.5)
- moved C24 54.3 mm to (148.3, 44.7), turned to 270 degrees
- moved R3 52.3 mm to (124.0, 43.4)
- moved R2 51.6 mm to (101.1, 63.2)
- moved C21 51.1 mm to (146.6, 44.5), turned to 270 degrees
- moved R10 51.0 mm to (136.1, 35.6), turned to 180 degrees
- moved R11 50.3 mm to (147.6, 41.4)
- moved J3 49.9 mm to (160.5, 101.1), turned to 270 degrees
- moved FB4 47.0 mm to (137.7, 52.8), turned to 180 degrees
- moved R8 47.0 mm to (100.8, 69.1)
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Connections:
- J4 pad 39: +3V3 -> Net-(J4-Pad39)
- J4 pad 40: +3V3 -> Net-(J4-Pad39)
- U1 pad 3: +3V3 -> +5V
- U2 pad 3: +3V3 -> +5V
Other:
- board text added: "1.9V"
- board text added: "3.3V"
- board text added: "3.3V In"
- board text added: "3.3V Local"

Commit message: Misc missed changes? Been a while since I really looked
Parts:
- added C31: 10u, Capacitor_SMD:C_0805_2012Metric_Pad1.18x1.45mm_HandSolder, F.Cu at (105.7, 58.9)
- added C32: 10u, Capacitor_SMD:C_0805_2012Metric_Pad1.18x1.45mm_HandSolder, F.Cu at (105.2, 67.8)
- added C33: 10u, Capacitor_SMD:C_0805_2012Metric_Pad1.18x1.45mm_HandSolder, F.Cu at (104.9, 77.7)
- R1, R17, R8: value R -> 10k
- R18: value R -> 12k
- R2, R9: value R -> 3.6k
